File: Projects/Sketch/breakout.sch (KiCad schematic (older format))
At the start: 37 parts, among them J1 JACK_TRS_4PINS, P1 CONN_01X08, P2 SPEAKER, P3 ISO7816_SIMPLE, P4 CONN_01X09, P5 SMA_CONN, P6 MIC, P7 USB_OTG, Q1 Q_PMOS_GSD, Q2 Q_NMOS_GSD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

Commit message: Update 23 Desember 2019 (Menambah Video & Sketch Eagle)
Parts:
- C1, C10, C11, C2, C5, C6, C7, C8, C9: symbol C -> Device:C
- C3: symbol CP -> Device:CP
- C4: symbol C_Small -> Device:C_Small
- D1: symbol LED-RESCUE-breakout -> breakout-rescue:LED-RESCUE-breakout
- GSM1: symbol A6_GSM -> breakout-rescue:A6_GSM
- J1: symbol JACK_TRS_4PINS -> breakout-rescue:JACK_TRS_4PINS
- L1, L2, L3, L4: symbol L_Small -> Device:L_Small
- P1: symbol CONN_01X08 -> breakout-rescue:CONN_01X08
- P2, P5, P6: symbol CONN_01X02 -> breakout-rescue:CONN_01X02
- P3: symbol ISO7816_SIMPLE -> breakout-rescue:ISO7816_SIMPLE
- P4: symbol CONN_01X09 -> breakout-rescue:CONN_01X09
- P7: symbol USB_OTG-RESCUE-breakout -> breakout-rescue:USB_OTG-RESCUE-breakout
- Q1: symbol Q_PMOS_GSD -> Device:Q_PMOS_GSD
- Q2: symbol Q_NMOS_GSD -> Device:Q_NMOS_GSD
- R1, R2, R3, R4, R5, R6, R7, R8: symbol R -> Device:R
- U1: symbol APE8865Y5-31-HF-3-RESCUE-breakout -> breakout-rescue:APE8865Y5-31-HF-3-RESCUE-breakout
- U2: symbol ESP-12E -> breakout-rescue:ESP-12E
