File: Projects/Sketch/KAnggara75/KAnggara75.brd (EAGLE design)
At the start: 160 x 100 mm, 34 parts, among them IC1 LM1117MPX-3.3, Q1 SS8050-G, Q2 SS8050-G, U1 CP2102N-A01-GQFN28, U2 ESP-WROOM-32, X1 ZX62D-B-5PA8

Commit message: Update 1 Januari 2020
Parts:
- added C10, C11, C12: 0.1u, rcl:C0805
- added D5, D6, D7: (no value), diode:P2-15
- added D8: BAT60J, diode:SOD323_ST
- added IC2: HT7333, holtek2:SOT-89
- added IC3: TP4056, TP4056:SOP-8
- added JP2: (no value), pinhead:1X02
- added LED2: Blue, led:1206
- added LED3: Red, led:1206
- added R11, R12, R14: 1k, rcl:R0805
- added R13: 1.2k, rcl:R0805
- added R15: 100, rcl:R0805
- added T1: DMN3024LSD, FS8205A:TSSOP-8
- added U$2: BATTERY-LI-MH12210, diy-modules:BATTERY-LI-MH12210
- added U$3: U-BLOX-NEO6V2, u-blox neo-6m v2:U-BLOX-NEO6V2
- added U$5: DW01A, DW01A:SOT23-6
- added X2: ZX62D-B-5PA8, zx62d-b-5pa8-oshpark_10:ZX62D-B-5PA8
- moved C9 204.8 mm to (-55.9, 104.1)
- moved C8 196.2 mm to (-49.5, 96.5)
- moved R7 184.3 mm to (-33.0, 96.5)
- moved C7 181.8 mm to (-40.6, 104.1)
- moved R8 178.6 mm to (-40.6, 88.9)
- moved R9 177.9 mm to (-50.8, 88.9)
- moved Q2 168.4 mm to (-72.4, 109.2)
- moved S2 167.7 mm to (-30.5, 78.7)
- moved Q1 167.5 mm to (-63.5, 109.2)
- moved C6 167.1 mm to (-25.4, 104.1)
- moved R10 164.7 mm to (-86.4, 88.9)
- moved C5 160.3 mm to (-80.0, 96.5)
- moved D4 158.6 mm to (-47.0, 110.5)
- moved R4 158.2 mm to (-25.4, 96.5)
- moved R3 157.5 mm to (-17.8, 96.5)
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Connections:
- new net BAT+: C12.1, IC2.3, IC2.4, R15.1, U$2.BAT+
- new net BAT-: C11.2, IC2.2, T1.6, T1.7, U$2.BAT-, U$5.6
- new net IN+: C10.1, IC3.4, JP2.2, LED2.A, LED3.A
- new net IN-: C10.2, C12.2, IC3.1, IC3.3, JP2.1, R13.1, R14.1, T1.2, T1.3
- new net N$10: U$3.VCC
- new net N$11: LED3.C, R12.1
- new net N$12: IC3.6, R11.2
- new net N$13: IC3.7, R12.2
- new net N$15: T1.1, T1.8
- new net N$16: T1.4, U$5.3
- new net N$17: T1.5, U$5.1
- new net N$18: IC3.2, R13.2
- new net N$19: R14.2, U$5.2
- new net N$20: C11.1, R15.2, U$5.5
- new net N$7: LED2.C, R11.1
- new net N$8: U$3.TX
- new net N$9: U$3.RX
- new net OUT+: IC3.5
- net D+: now also D7.C, X2.3
- net D-: now also D6.C, X2.2
- net GND: now also U$3.GND
- net PE: now also D5.A, D6.A, D7.A, X2.5
- net VCC: now also D8.C, IC2.1
- net VEE: now also D5.C, D8.A, X2.1
Routing:
- net IN-: track 0.00 -> 84.2 mm
- net IN+: track 0.00 -> 55.9 mm
- net BAT-: track 0.00 -> 20.7 mm
- net N$20: track 0.00 -> 17.1 mm
- net BAT+: track 0.00 -> 12.1 mm
- net N$18: track 0.00 -> 6.36 mm
- net N$16: track 0.00 -> 5.75 mm
- net N$13: track 0.00 -> 4.67 mm
- net N$12: track 0.00 -> 4.67 mm
- net N$7: track 0.00 -> 4.47 mm
- net N$11: track 0.00 -> 4.47 mm

Commit message: Make Folder Project ESP32
Parts:
- moved X1 68.9 mm to (0.77, 35.5)
Changed lines of the file:
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@@
 </element>
 <element name="U2" library="esp32" package="ESP-WROOM-32" value="ESP-WROOM-32" x="86.24" y="88.86" rot="R270"/>
-<element name="X1" library="zx62d-b-5pa8-oshpark_10" package="ZX62D-B-5PA8" value="ZX62D-B-5PA8" x="-62.23" y="63.5">
-<attribute name="MF" value="Hirose" x="-62.23" y="63.5" size="1.778" layer="27" display="off"/>
-<attribute name="OC_NEWARK" value="69W0712" x="-62.23" y="63.5" size="1.778" layer="27" display="off"/>
-<attribute name="MPN" value="ZX62D-B-5PA8" x="-62.23" y="63.5" size="1.778" layer="27" display="off"/>
-<attribute name="OC_FARNELL" value="2300438" x="-62.23" y="63.5" size="1.778" layer="27" display="off"/>
+<element name="X1" library="zx62d-b-5pa8-oshpark_10" package="ZX62D-B-5PA8" value="ZX62D-B-5PA8" x="0.77" y="35.5">
+<attribute name="MF" value="Hirose" x="0.77" y="35.5" size="1.778" layer="27" display="off"/>
+<attribute name="OC_NEWARK" value="69W0712" x="0.77" y="35.5" size="1.778" layer="27" display="off"/>
+<attribute name="MPN" value="ZX62D-B-5PA8" x="0.77" y="35.5" size="1.778" layer="27" display="off"/>
+<attribute name="OC_FARNELL" value="2300438" x="0.77" y="35.5" size="1.778" layer="27" display="off"/>
 </element>
 <element name="U$3" library="u-blox neo-6m v2" package="U-BLOX-NEO6V2" value="U-BLOX-NEO6V2" x="4" y="78" rot="R270"/>
@@
 <wire x1="-90.62" y1="-56" x2="-59.75" y2="-93" width="0" layer="19" extent="1-1"/>
 <wire x1="-88.175" y1="-27.7" x2="-90.62" y2="-56" width="0" layer="19" extent="1-1"/>
-<wire x1="-57.405" y1="64.8" x2="-88.175" y2="-27.7" width="0" layer="19" extent="1-1"/>
-<wire x1="-62.23" y1="77.47" x2="-57.405" y2="64.8" width="0" layer="19" extent="1-1"/>
+<wire x1="5.595" y1="36.8" x2="-88.175" y2="-27.7" width="0" layer="19" extent="1-1"/>
+<wire x1="-62.23" y1="77.47" x2="5.595" y2="36.8" width="0" layer="19" extent="1-1"/>
 <wire x1="-45.74" y1="110.49" x2="-62.23" y2="77.47" width="0" layer="19" extent="1-1"/>
-<wire x1="-15.06" y1="59.95" x2="-57.405" y2="64.8" width="0" layer="19" extent="1-1"/>
+<wire x1="-15.06" y1="59.95" x2="5.595" y2="36.8" width="0" layer="19" extent="1-1"/>
 <wire x1="-15.06" y1="58.55" x2="-15.06" y2="59.95" width="0" layer="19" extent="1-1"/>
 </signal>
@@
 <wire x1="-81.1" y1="61.46" x2="-78.74" y2="60.96" width="0" layer="19" extent="1-1"/>
 <wire x1="-67.31" y1="77.47" x2="-78.74" y2="60.96" width="0" layer="19" extent="1-1"/>
-<wire x1="-57.405" y1="62.2" x2="-67.31" y2="77.47" width="0" layer="19" extent="1-1"/>
-<wire x1="-46.99" y1="77.47" x2="-57.405" y2="62.2" width="0" layer="19" extent="1-1"/>
+<wire x1="5.595" y1="34.2" x2="-67.31" y2="77.47" width="0" layer="19" extent="1-1"/>
+<wire x1="-46.99" y1="77.47" x2="5.595" y2="34.2" width="0" layer="19" extent="1-1"/>
 <wire x1="-33.7312" y1="76.4794" x2="-46.99" y2="77.47" width="0" layer="19" extent="1-1"/>
 <wire x1="-27.2288" y1="76.4794" x2="-33.7312" y2="76.4794" width="0" layer="19" extent="1-1"/>
@@
 <wire x1="-88.175" y1="-29" x2="-90.62" y2="-102" width="0" layer="19" extent="1-1"/>
 <wire x1="-81.1" y1="60.96" x2="-88.175" y2="-29" width="0" layer="19" extent="1-1"/>
-<wire x1="-57.405" y1="63.5" x2="-81.1" y2="60.96" width="0" layer="19" extent="1-1"/>
-<wire x1="-30.48" y1="87.63" x2="-57.405" y2="63.5" width="0" layer="19" extent="1-1"/>
+<wire x1="5.595" y1="35.5" x2="-81.1" y2="60.96" width="0" layer="19" extent="1-1"/>
+<wire x1="-30.48" y1="87.63" x2="5.595" y2="35.5" width="0" layer="19" extent="1-1"/>
 </signal>
 <signal name="D-">
@@
 <wire x1="-81.1" y1="60.46" x2="-88.175" y2="-28.35" width="0" layer="19" extent="1-1"/>
 <wire x1="-82.55" y1="77.47" x2="-81.1" y2="60.46" width="0" layer="19" extent="1-1"/>
-<wire x1="-57.405" y1="64.15" x2="-81.1" y2="60.46" width="0" layer="19" extent="1-1"/>
+<wire x1="5.595" y1="36.15" x2="-81.1" y2="60.46" width="0" layer="19" extent="1-1"/>
 </signal>
 <signal name="RXD">
