File: Projects/Sketch/KAnggara75/KAnggara75.sch (EAGLE design)
At the start: 34 parts, among them IC1 LM1117MPX-3.3, Q1 SS8050-G, Q2 SS8050-G, U1 CP2102N-A01-GQFN28, U2 ESP-WROOM-32, X1 ZX62D-B-5PA8

Commit message: Update 1 Januari 2020
Parts:
- added C10, C11, C12: 0.1u, rcl:C-EUC0805
- added D5, D6, D7: (no value), diode:DIODE_SCHOTTKY2-P2-15
- added D8: BAT60J, diode:BAT60J
- added IC2: HT7333, holtek2:HT7333
- added IC3: TP4056, TP4056:TP4056
- added JP2: (no value), pinhead:PINHD-1X2
- added LED2: Blue, led:LEDSMT1206
- added LED3: Red, led:LEDSMT1206
- added R11, R12, R14: 1k, rcl:R-EU_R0805
- added R13: 1.2k, rcl:R-EU_R0805
- added R15: 100, rcl:R-EU_R0805
- added T1: DMN3024LSD, FS8205A:DMN3024LSD
- added U$2: BATTERY-LI-MH12210, diy-modules:BATTERY-LI-MH12210
- added U$3: U-BLOX-NEO6V2, u-blox neo-6m v2:U-BLOX-NEO6V2
- added U$5: DW01A, DW01A:DW01A
- added X2: ZX62D-B-5PA8, zx62d-b-5pa8-oshpark_10:ZX62D-B-5PA8
Connections:
- new net BAT+: C12.1, IC2.IN, R15.1, U$2.BAT+
- new net BAT-: C11.2, IC2.GND, T1B.S, U$2.BAT-, U$5.GND
- new net IN+: C10.1, IC3.VCC, JP2.2, LED2.A, LED3.A
- new net IN-: C10.2, C12.2, IC3.GND, IC3.TEMP, JP2.1, R13.1, R14.1, T1A.S
- new net N$10: U$3.VCC
- new net N$11: LED3.C, R12.1
- new net N$12: IC3.STDBY, R11.2
- new net N$13: IC3.CHRG, R12.2
- new net N$15: T1A.D, T1B.D
- new net N$16: T1A.G, U$5.OC
- new net N$17: T1B.G, U$5.OD
- new net N$18: IC3.PROG, R13.2
- new net N$19: R14.2, U$5.CS
- new net N$20: C11.1, R15.2, U$5.VCC
- new net N$7: LED2.C, R11.1
- new net N$8: U$3.TX
- new net N$9: U$3.RX
- new net OUT+: IC3.BAT
- net D+: now also D7.2, X2G$1.3
- net D-: now also D6.2, X2G$1.2
- net GND: now also U$3.GND
- net PE: now also D5.1, D6.1, D7.1, X2G$1.5
- net VCC: now also D8.C, IC2.OUT
- net VEE: now also D5.2, D8.A, X2G$1.1

Commit message: Make Folder Project ESP32
Changed lines of the file:
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@@
 <?xml version="1.0" encoding="utf-8"?>
 <!DOCTYPE eagle SYSTEM "eagle.dtd">
-<eagle version="7.7.0">
+<eagle version="9.5.2">
 <drawing>
 <settings>
 <setting alwaysvectorfont="no"/>
+<setting keepoldvectorfont="yes"/>
 <setting verticaltext="up"/>
 </settings>
-<grid distance="0.1" unitdist="inch" unit="inch" style="lines" multiple="1" display="yes" altdistance="0.01" altunitdist="inch" altunit="inch"/>
+<grid distance="0.1" unitdist="inch" unit="inch" style="lines" multiple="1" display="no" altdistance="0.01" altunitdist="inch" altunit="inch"/>
 <layers>
 <layer number="1" name="Top" color="4" fill="1" visible="no" active="no"/>
@@
 <attribute name="VALUE" x="567.055" y="140.081" size="1.778" layer="96"/>
 </instance>
-<instance part="FRAME2" gate="G$1" x="0" y="0"/>
-<instance part="U$3" gate="G$1" x="596.9" y="294.64"/>
+<instance part="FRAME2" gate="G$1" x="0" y="0" smashed="yes">
+<attribute name="DRAWING_NAME" x="217.17" y="15.24" size="2.54" layer="94"/>
+<attribute name="LAST_DATE_TIME" x="217.17" y="10.16" size="2.286" layer="94"/>
+<attribute name="SHEET" x="230.505" y="5.08" size="2.54" layer="94"/>
+</instance>
+<instance part="U$3" gate="G$1" x="596.9" y="294.64" smashed="yes"/>
 </instances>
 <busses>
@@
 </plain>
 <instances>
-<instance part="FRAME1" gate="G$1" x="0" y="0"/>
-<instance part="U$2" gate="G$1" x="27.94" y="157.48"/>
-<instance part="IC2" gate="G$1" x="15.24" y="144.78"/>
-<instance part="X2" gate="G$1" x="99.06" y="165.1" rot="R90"/>
+<instance part="FRAME1" gate="G$1" x="0" y="0" smashed="yes">
+<attribute name="DRAWING_NAME" x="217.17" y="15.24" size="2.54" layer="94"/>
+<attribute name="LAST_DATE_TIME" x="217.17" y="10.16" size="2.286" layer="94"/>
+<attribute name="SHEET" x="230.505" y="5.08" size="2.54" layer="94"/>
+</instance>
+<instance part="U$2" gate="G$1" x="27.94" y="157.48" smashed="yes">
+<attribute name="NAME" x="12.7" y="170.18" size="1.778" layer="95"/>
+<attribute name="VALUE" x="12.7" y="167.64" size="1.778" layer="96"/>
+</instance>
+<instance part="IC2" gate="G$1" x="15.24" y="144.78" smashed="yes">
+<attribute name="NAME" x="17.78" y="137.16" size="1.778" layer="95"/>
+<attribute name="VALUE" x="17.78" y="134.62" size="1.778" layer="96"/>
+</instance>
+<instance part="X2" gate="G$1" x="99.06" y="165.1" smashed="yes" rot="R90">
+<attribute name="NAME" x="87.63" y="162.56" size="1.778" layer="95" font="vector" rot="R90"/>
+<attribute name="VALUE" x="106.68" y="173.99" size="1.778" layer="96" font="vector" rot="R180"/>
+</instance>
 <instance part="SUPPLY17" gate="G$1" x="91.44" y="154.94" smashed="yes" rot="R90">
 <attribute name="VALUE" x="88.265" y="153.035" size="1.778" layer="96" rot="R90"/>
@@
 <attribute name="VALUE" x="125.095" y="150.495" size="1.778" layer="96"/>
 </instance>
-<instance part="IC3" gate="G$1" x="40.64" y="96.52"/>
-<instance part="U$5" gate="G$1" x="93.98" y="106.68" rot="MR0"/>
-<instance part="LED2" gate="G$1" x="15.24" y="91.44" rot="R180"/>
-<instance part="LED3" gate="G$1" x="25.4" y="91.44" rot="R180"/>
-<instance part="R11" gate="G$1" x="15.24" y="104.14" rot="R90"/>
-<instance part="R12" gate="G$1" x="25.4" y="104.14" rot="R90"/>
-<instance part="T1" gate="A" x="81.28" y="83.82" rot="R270"/>
-<instance part="T1" gate="B" x="91.44" y="83.82" rot="MR270"/>
-<instance part="R13" gate="G$1" x="33.02" y="83.82" rot="R90"/>
-<instance part="C10" gate="G$1" x="22.86" y="83.82"/>
-<instance part="R14" gate="G$1" x="73.66" y="93.98" rot="R90"/>
-<instance part="C11" gate="G$1" x="106.68" y="106.68"/>
-<instance part="R15" gate="G$1" x="116.84" y="109.22" rot="R180"/>
-<instance part="C12" gate="G$1" x="121.92" y="91.44"/>
-<instance part="JP2" gate="G$1" x="7.62" y="66.04" rot="R180"/>
+<instance part="IC3" gate="G$1" x="40.64" y="96.52" smashed="yes">
+<attribute name="NAME" x="40.64" y="96.52" size="1.27" layer="95"/>
+<attribute name="VALUE" x="40.64" y="81.28" size="1.27" layer="96"/>
+</instance>
+<instance part="U$5" gate="G$1" x="93.98" y="106.68" smashed="yes" rot="MR0"/>
+<instance part="LED2" gate="G$1" x="15.24" y="91.44" smashed="yes" rot="R180">
+<attribute name="NAME" x="11.684" y="96.012" size="1.778" layer="95" rot="R270"/>
+<attribute name="VALUE" x="9.525" y="96.012" size="1.778" layer="96" rot="R270"/>
+</instance>
+<instance part="LED3" gate="G$1" x="25.4" y="91.44" smashed="yes" rot="R180">
+<attribute name="NAME" x="21.844" y="96.012" size="1.778" layer="95" rot="R270"/>
+<attribute name="VALUE" x="19.685" y="96.012" size="1.778" layer="96" rot="R270"/>
+</instance>
+<instance part="R11" gate="G$1" x="15.24" y="104.14" smashed="yes" rot="R90">
+<attribute name="NAME" x="13.7414" y="100.33" size="1.778" layer="95" rot="R90"/>
+<attribute name="VALUE" x="18.542" y="100.33" size="1.778" layer="96" rot="R90"/>
+</instance>
+<instance part="R12" gate="G$1" x="25.4" y="104.14" smashed="yes" rot="R90">
+<attribute name="NAME" x="23.9014" y="100.33" size="1.778" layer="95" rot="R90"/>
+<attribute name="VALUE" x="28.702" y="100.33" size="1.778" layer="96" rot="R90"/>
+</instance>
+<instance part="T1" gate="A" x="81.28" y="83.82" smashed="yes" rot="R270">
+<attribute name="VALUE" x="81.28" y="81.28" size="1.778" layer="96" rot="R270"/>
+<attribute name="NAME" x="83.82" y="81.28" size="1.778" layer="95" rot="R270"/>
+</instance>
+<instance part="T1" gate="B" x="91.44" y="83.82" smashed="yes" rot="MR270">
+<attribute name="VALUE" x="91.44" y="81.28" size="1.778" layer="96" rot="MR270"/>
+<attribute name="NAME" x="88.9" y="81.28" size="1.778" layer="95" rot="MR270"/>
+</instance>
+<instance part="R13" gate="G$1" x="33.02" y="83.82" smashed="yes" rot="R90">
+<attribute name="NAME" x="31.5214" y="80.01" size="1.778" layer="95" rot="R90"/>
+<attribute name="VALUE" x="36.322" y="80.01" size="1.778" layer="96" rot="R90"/>
+</instance>
+<instance part="C10" gate="G$1" x="22.86" y="83.82" smashed="yes">
+<attribute name="NAME" x="24.384" y="84.201" size="1.778" layer="95"/>
+<attribute name="VALUE" x="24.384" y="79.121" size="1.778" layer="96"/>
+</instance>
+<instance part="R14" gate="G$1" x="73.66" y="93.98" smashed="yes" rot="R90">
+<attribute name="NAME" x="72.1614" y="90.17" size="1.778" layer="95" rot="R90"/>
+<attribute name="VALUE" x="76.962" y="90.17" size="1.778" layer="96" rot="R90"/>
+</instance>
+<instance part="C11" gate="G$1" x="106.68" y="106.68" smashed="yes">
+<attribute name="NAME" x="108.204" y="107.061" size="1.778" layer="95"/>
+<attribute name="VALUE" x="108.204" y="101.981" size="1.778" layer="96"/>
+</instance>
+<instance part="R15" gate="G$1" x="116.84" y="109.22" smashed="yes" rot="R180">
+<attribute name="NAME" x="120.65" y="107.7214" size="1.778" layer="95" rot="R180"/>
+<attribute name="VALUE" x="120.65" y="112.522" size="1.778" layer="96" rot="R180"/>
+</instance>
+<instance part="C12" gate="G$1" x="121.92" y="91.44" smashed="yes">
+<attribute name="NAME" x="123.444" y="91.821" size="1.778" layer="95"/>
+<attribute name="VALUE" x="123.444" y="86.741" size="1.778" layer="96"/>
+</instance>
+<instance part="JP2" gate="G$1" x="7.62" y="66.04" smashed="yes" rot="R180">
+<attribute name="NAME" x="13.97" y="60.325" size="1.778" layer="95" rot="R180"/>
+<attribute name="VALUE" x="13.97" y="71.12" size="1.778" layer="96" rot="R180"/>
+</instance>
 </instances>
 <busses>
@@
 </nets>
 </sheet>
+<sheet>
+<description>KL</description>
+<plain>
+</plain>
+<instances>
+</instances>
+<busses>
+</busses>
+<nets>
+</nets>
+</sheet>
