File: Projects/TheSiS_HW/TheSiS.brd (EAGLE design)
At the start: 92.7 x 98.7 mm, 80 parts, among them IC1 REG1117, IC3 TP4056, IC4 MCP1703CB, IC5 CP2102, K1 G5L, K2 G5L, K3 G5L, T1 DMN3024LSD, U1 ESP-WROOM-32, U2 GY-521MPU6050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

Commit message: Menamahkan Logo
Parts:
- moved C1 40.4 mm to (76.1, 104.0)
- moved C12 40.4 mm to (48.3, 85.1)
- moved C13 40.4 mm to (42.3, 105.0)
- moved C14 40.4 mm to (42.3, 97.4)
- moved C2 40.4 mm to (77.9, 108.8)
- moved C4 40.4 mm to (60.1, 93.0)
- moved C5 40.4 mm to (44.9, 86.0)
- moved C6 40.4 mm to (44.9, 80.9)
- moved D1 40.4 mm to (57.6, 88.5)
- moved D2 40.4 mm to (74.7, 26.3)
- moved D3 40.4 mm to (76.0, 33.4)
- moved IC1 40.4 mm to (59.8, 81.3)
- moved IC4 40.4 mm to (65.9, 93.0)
- moved IC5 40.4 mm to (52.5, 75.8)
- moved LED1 40.4 mm to (61.4, 108.8)
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
Commit message: Finish Hardware v20.10.21
Parts:
- moved LED3 1.02 mm to (63.0, 87.6), turned to 270 degrees
- renumbered U$2 to 18650
Connections:
- new net EXT5V: C4.1, D1.C, IC1.3, R4.2
- net VIN5V: no longer C4.1, D1.C, IC1.3, R4.2
Routing:
- net EXT5V: track 0.00 -> 8.85 mm
- net VIN5V: track 73.4 -> 65.3 mm
- net GND: track 382.4 -> 381.5 mm
- net N$10: track 2.58 -> 1.88 mm
- added copper zone on layer 1, net GND
- added copper zone on layer 16, net GND
Other:
- board size 92.7 x 98.7 mm -> 92.3 x 99.4 mm

Commit message: Finish Board v20.10.20 [Order PCBWay.com]
Parts:
- removed U2: GY-521MPU6050, gy-521:GY-521
- added JP1, SV1: (no value), pinhead:1X04
- added U$2: (no value), holes:3,0
- U$3: value U-BLOX-NEO6V2 -> (none); device u-blox neo-6m v2:U-BLOX-NEO6V2 -> holes:3,0
- moved U$3 39.6 mm to (122.4, 42.5), turned to 0 degrees
Connections:
- removed net N$33: S2.4, U2.VCC
- removed net N$37: U2.XDA
- removed net N$38: U2.XCL
- removed net N$39: U2.ADO
- removed net N$40: U2.INT
- new net N$35: JP1.1, S2.4
- net BAT+: now also SV1.1; no longer U$3.VCC
- net GND: now also JP1.2, SV1.4; no longer U$3.GND, U2.GND
- net IO16: now also SV1.3; no longer U$3.TX
- net IO17: now also SV1.2; no longer U$3.RX
- net IO21: now also JP1.4; no longer U2.SDA
- net IO22: now also JP1.3; no longer U2.SCL
Routing:
- net N$33: track 60.0 -> 0.00 mm
- net N$35: track 0.00 -> 59.8 mm
- net GND: track 381.5 -> 369.1 mm, vias 16 -> 15
- net BAT+: track 232.1 -> 223.0 mm
- net IO16: track 45.2 -> 42.3 mm
- net IO17: track 44.5 -> 41.5 mm
- net IO22: track 10.1 -> 7.21 mm, vias 1 -> 0
- net IO21: track 9.57 -> 7.70 mm
Other:
- board size 92.3 x 99.4 mm -> 92.2 x 99.2 mm

Commit message: Sebelum install November 2020
Parts:
- IC1: device burr-brown:SOT223 -> REG1117:SOT223A
- IC5: device silabs:MLP28 -> CP2102:QFN28
- K1, K2, K3: value G5L -> G5LE; device relay:G5LE -> G5LE_1:G5LE
- OK1, OK2, OK3: device optocoupler:MINI-FLAT-4 -> tlp283:SOT23-4
- X1, X3, X4: device con-wago-508:W237-133 -> Terminal_Block_5mm.:W237-3
Routing:
- net N$35: track 59.8 -> 56.0 mm
- net N$22: track 12.5 -> 8.67 mm
- net IO04: track 124.1 -> 120.3 mm
- net IO02: track 132.8 -> 129.0 mm
