File: Projects/TheSiS_HW/TheSiS.sch (EAGLE design)
At the start: 80 parts, among them IC1 REG1117, IC3 TP4056, IC4 MCP1703CB, IC5 CP2102, K1 G5L, K2 G5L, K3 G5L, T1 DMN3024LSD, U1 ESP-WROOM-32, X2 ZX62D-B-5PA8

Commit message: Sebelum install November 2020
Parts:
- IC1: device burr-brown:REG1117 -> REG1117:REG1117
- IC5: device silabs:CP2102 -> CP2102:CP2102
- K1, K2, K3: value G5L -> G5LE; device relay:G5L -> G5LE_1:G5LE
- OK1, OK2, OK3: device optocoupler:TLP283 -> tlp283:TLP283
- X1, X3, X4: device con-wago-508:W237-03P -> Terminal_Block_5mm.:W237-03P
Changed lines of the file:
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@@
 </groups>
 <parts>
-<part name="U1" library="esp32" deviceset="ESP-WROOM-32" device=""/>
+<part name="U1" library="esp32" library_urn="urn:adsk.eagle:library:24322740" deviceset="ESP-WROOM-32" device="" package3d_urn="urn:adsk.eagle:package:24322748/2"/>
 <part name="FRAME1" library="frames" library_urn="urn:adsk.eagle:library:229" deviceset="A3L-LOC" device=""/>
-<part name="IC1" library="burr-brown" library_urn="urn:adsk.eagle:library:111" deviceset="REG1117" device="" package3d_urn="urn:adsk.eagle:package:4940/1"/>
+<part name="IC1" library="REG1117" library_urn="urn:adsk.eagle:library:24332741" deviceset="REG1117" device="" package3d_urn="urn:adsk.eagle:package:24332763/2"/>
 <part name="SUPPLY2" library="supply2" library_urn="urn:adsk.eagle:library:372" deviceset="GND" device=""/>
 <part name="SUPPLY5" library="supply2" library_urn="urn:adsk.eagle:library:372" deviceset="GND" device=""/>
 <part name="S1" library="switch-dil" library_urn="urn:adsk.eagle:library:375" deviceset="DIP04S" device="" package3d_urn="urn:adsk.eagle:package:27250/2"/>
 <part name="S2" library="switch-dil" library_urn="urn:adsk.eagle:library:375" deviceset="DIP08S" device="" package3d_urn="urn:adsk.eagle:package:27257/2"/>
-<part name="U$1" library="DW01A" deviceset="DW01A" device=""/>
+<part name="U$1" library="DW01A" library_urn="urn:adsk.eagle:library:24332452" deviceset="DW01A" device="" package3d_urn="urn:adsk.eagle:package:24332455/2"/>
 <part name="18650" library="diy-modules" deviceset="BATTERY-LI-MH12210" device=""/>
-<part name="T1" library="FS8205A" deviceset="DMN3024LSD" device=""/>
-<part name="IC3" library="TP4056" deviceset="TP4056" device=""/>
+<part name="T1" library="FS8205A" library_urn="urn:adsk.eagle:library:24332876" deviceset="DMN3024LSD" device="" package3d_urn="urn:adsk.eagle:package:24332881/2"/>
+<part name="IC3" library="TP4056" library_urn="urn:adsk.eagle:library:24322954" deviceset="TP4056" device="" package3d_urn="urn:adsk.eagle:package:24322957/2"/>
 <part name="SUPPLY6" library="supply2" library_urn="urn:adsk.eagle:library:372" deviceset="GND" device=""/>
 <part name="R1" library="rcl" library_urn="urn:adsk.eagle:library:334" deviceset="R-EU_" device="R0603" package3d_urn="urn:adsk.eagle:package:23555/3" value="1k"/>
@@
 <part name="R10" library="rcl" library_urn="urn:adsk.eagle:library:334" deviceset="R-EU_" device="R0805" package3d_urn="urn:adsk.eagle:package:23553/2" value="100k"/>
 <part name="C9" library="rcl" library_urn="urn:adsk.eagle:library:334" deviceset="C-EU" device="C0805" package3d_urn="urn:adsk.eagle:package:23617/2" value="22µ"/>
-<part name="D1" library="BAT760-7" deviceset="BAT760-7" device=""/>
-<part name="IC5" library="silabs" library_urn="urn:adsk.eagle:library:358" deviceset="CP210*" device="" package3d_urn="urn:adsk.eagle:package:26377/1" technology="2"/>
+<part name="D1" library="BAT760-7" library_urn="urn:adsk.eagle:library:24332698" deviceset="BAT760-7" device="" package3d_urn="urn:adsk.eagle:package:24332701/2"/>
+<part name="IC5" library="CP2102" library_urn="urn:adsk.eagle:library:24332818" deviceset="CP210*" device="" package3d_urn="urn:adsk.eagle:package:24332836/2" technology="2"/>
 <part name="SUPPLY9" library="supply2" library_urn="urn:adsk.eagle:library:372" deviceset="GND" device=""/>
 <part name="R7" library="rcl" library_urn="urn:adsk.eagle:library:334" deviceset="R-EU_" device="R0805" package3d_urn="urn:adsk.eagle:package:23553/2" value="22.1k"/>
@@
 <part name="SUPPLY3" library="supply2" library_urn="urn:adsk.eagle:library:372" deviceset="GND" device=""/>
 <part name="SUPPLY4" library="supply2" library_urn="urn:adsk.eagle:library:372" deviceset="GND" device=""/>
-<part name="U$4" library="sim800l" deviceset="SIM800L" device=""/>
-<part name="K3" library="relay" library_urn="urn:adsk.eagle:library:339" deviceset="G5L" device="" package3d_urn="urn:adsk.eagle:package:24308/1"/>
+<part name="U$4" library="sim800l" library_urn="urn:adsk.eagle:library:24332850" deviceset="SIM800L" device="" package3d_urn="urn:adsk.eagle:package:24332856/2"/>
+<part name="K3" library="G5LE_1" library_urn="urn:adsk.eagle:library:24325471" deviceset="G5LE" device="" package3d_urn="urn:adsk.eagle:package:24324955/3"/>
 <part name="R18" library="rcl" library_urn="urn:adsk.eagle:library:334" deviceset="R-EU_" device="R0805" package3d_urn="urn:adsk.eagle:package:23553/2" value="220"/>
 <part name="R19" library="rcl" library_urn="urn:adsk.eagle:library:334" deviceset="R-EU_" device="R0805" package3d_urn="urn:adsk.eagle:package:23553/2" value="10k"/>
@@
 <part name="D2" library="diode" library_urn="urn:adsk.eagle:library:210" deviceset="PMLL41*" device="SOD80C" package3d_urn="urn:adsk.eagle:package:43405/2"/>
 <part name="LED4" library="led" library_urn="urn:adsk.eagle:library:259" deviceset="LED" device="CHIP-LED0805" package3d_urn="urn:adsk.eagle:package:15818/2"/>
-<part name="OK2" library="optocoupler" library_urn="urn:adsk.eagle:library:320" deviceset="TLP283" device="" package3d_urn="urn:adsk.eagle:package:21958/1"/>
-<part name="X1" library="con-wago-508" library_urn="urn:adsk.eagle:library:196" deviceset="W237-03P" device="" package3d_urn="urn:adsk.eagle:package:10737/1"/>
-<part name="K1" library="relay" library_urn="urn:adsk.eagle:library:339" deviceset="G5L" device="" package3d_urn="urn:adsk.eagle:package:24308/1"/>
+<part name="OK2" library="tlp283" library_urn="urn:adsk.eagle:library:24332600" deviceset="TLP283" device="" package3d_urn="urn:adsk.eagle:package:24332653/2"/>
+<part name="X1" library="Terminal_Block_5mm." library_urn="urn:adsk.eagle:library:24333059" deviceset="W237-03P" device="" package3d_urn="urn:adsk.eagle:package:24333071/2"/>
+<part name="K1" library="G5LE_1" library_urn="urn:adsk.eagle:library:24325471" deviceset="G5LE" device="" package3d_urn="urn:adsk.eagle:package:24324955/3"/>
 <part name="R22" library="rcl" library_urn="urn:adsk.eagle:library:334" deviceset="R-EU_" device="R0805" package3d_urn="urn:adsk.eagle:package:23553/2" value="220"/>
 <part name="R23" library="rcl" library_urn="urn:adsk.eagle:library:334" deviceset="R-EU_" device="R0805" package3d_urn="urn:adsk.eagle:package:23553/2" value="10k"/>
@@
 <part name="D3" library="diode" library_urn="urn:adsk.eagle:library:210" deviceset="PMLL41*" device="SOD80C" package3d_urn="urn:adsk.eagle:package:43405/2"/>
 <part name="LED5" library="led" library_urn="urn:adsk.eagle:library:259" deviceset="LED" device="CHIP-LED0805" package3d_urn="urn:adsk.eagle:package:15818/2"/>
-<part name="OK1" library="optocoupler" library_urn="urn:adsk.eagle:library:320" deviceset="TLP283" device="" package3d_urn="urn:adsk.eagle:package:21958/1"/>
-<part name="X3" library="con-wago-508" library_urn="urn:adsk.eagle:library:196" deviceset="W237-03P" device="" package3d_urn="urn:adsk.eagle:package:10737/1"/>
-<part name="K2" library="relay" library_urn="urn:adsk.eagle:library:339" deviceset="G5L" device="" package3d_urn="urn:adsk.eagle:package:24308/1"/>
+<part name="OK1" library="tlp283" library_urn="urn:adsk.eagle:library:24332600" deviceset="TLP283" device="" package3d_urn="urn:adsk.eagle:package:24332653/2"/>
+<part name="X3" library="Terminal_Block_5mm." library_urn="urn:adsk.eagle:library:24333059" deviceset="W237-03P" device="" package3d_urn="urn:adsk.eagle:package:24333071/2"/>
+<part name="K2" library="G5LE_1" library_urn="urn:adsk.eagle:library:24325471" deviceset="G5LE" device="" package3d_urn="urn:adsk.eagle:package:24324955/3"/>
 <part name="R26" library="rcl" library_urn="urn:adsk.eagle:library:334" deviceset="R-EU_" device="R0805" package3d_urn="urn:adsk.eagle:package:23553/2" value="220"/>
 <part name="R27" library="rcl" library_urn="urn:adsk.eagle:library:334" deviceset="R-EU_" device="R0805" package3d_urn="urn:adsk.eagle:package:23553/2" value="10k"/>
@@
 <part name="D4" library="diode" library_urn="urn:adsk.eagle:library:210" deviceset="PMLL41*" device="SOD80C" package3d_urn="urn:adsk.eagle:package:43405/2"/>
 <part name="LED6" library="led" library_urn="urn:adsk.eagle:library:259" deviceset="LED" device="CHIP-LED0805" package3d_urn="urn:adsk.eagle:package:15818/2"/>
-<part name="OK3" library="optocoupler" library_urn="urn:adsk.eagle:library:320" deviceset="TLP283" device="" package3d_urn="urn:adsk.eagle:package:21958/1"/>
-<part name="X4" library="con-wago-508" library_urn="urn:adsk.eagle:library:196" deviceset="W237-03P" device="" package3d_urn="urn:adsk.eagle:package:10737/1"/>
+<part name="OK3" library="tlp283" library_urn="urn:adsk.eagle:library:24332600" deviceset="TLP283" device="" package3d_urn="urn:adsk.eagle:package:24332653/2"/>
+<part name="X4" library="Terminal_Block_5mm." library_urn="urn:adsk.eagle:library:24333059" deviceset="W237-03P" device="" package3d_urn="urn:adsk.eagle:package:24333071/2"/>
 <part name="JP1" library="pinhead" library_urn="urn:adsk.eagle:library:325" deviceset="PINHD-1X4" device="" package3d_urn="urn:adsk.eagle:package:22407/2"/>
 <part name="SV1" library="pinhead" library_urn="urn:adsk.eagle:library:325" deviceset="PINHD-1X4" device="" package3d_urn="urn:adsk.eagle:package:22407/2"/>
